File: universal_power_board/universal_power_board.sch (KiCad schematic (older format))
At the start: 25 parts, among them J1 Pixhawk Power, J10 5V OUTPUT, J11 BATT OUTPUT, J12 BATT OUTPUT, J2 BATT INPUT, J3 BATT OUTPUT, J4 5V OUTPUT, J5 5V OUTPUT, J6 BATT OUTPUT, J7 5V OUTPUT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

Commit message: update v1.1
Parts:
- C1: footprint Inductor_SMD:L_0603_1608Metric_Pad1.05x0.95mm_HandSolder -> Inductor_SMD:L_0805_2012Metric_Pad1.15x1.40mm_HandSolder
Connections:
- net +BATT: now also J11.2 (Pin_2), J12.2 (Pin_2), J3.2 (Pin_2), J6.2 (Pin_2); no longer J11.1 (Pin_1), J12.1 (Pin_1), J3.1 (Pin_1), J6.1 (Pin_1)
- net GND: now also J11.1 (Pin_1), J12.1 (Pin_1), J3.1 (Pin_1), J6.1 (Pin_1); no longer J11.2 (Pin_2), J12.2 (Pin_2), J3.2 (Pin_2), J6.2 (Pin_2)
Other:
- moved on the sheet: C2, J10, J2, J7, J8, J9
