File: universal_power_board_v1.2/universal_power_board_v1.2.sch (KiCad schematic (older format))
At the start: 25 parts, among them J1 Conn_01x03_Male, J10 5V OUTPUT, J11 BATT OUTPUT, J12 BATT OUTPUT, J2 BATT INPUT, J3 BATT OUTPUT, J4 5V OUTPUT, J5 5V OUTPUT, J6 BATT OUTPUT, J7 5V OUTPUT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

Commit message: v1.2プロジェクト作成
Changed lines of the file:
@@
 EESchema Schematic File Version 4
-LIBS:universal_power_board-cache
-EELAYER 29 0
+EELAYER 30 0
 EELAYER END
 $Descr A4 11693 8268
@@
 	1    0    0    -1
 $EndComp
-Wire Wire Line
-	2500 4600 2150 4600
-Wire Wire Line
-	2500 4800 2150 4800
 $Comp
 L Device:R_Small R1
@@
 Wire Wire Line
 	1700 4650 1700 4700
-Wire Wire Line
-	2500 4700 1700 4700
 Connection ~ 1700 4700
 Wire Wire Line
@@
 	5000 3500 5900 3500
 Wire Wire Line
+	2150 4800 2150 5050
+Wire Wire Line
 	2150 4400 2150 4600
-Wire Wire Line
-	2150 4800 2150 5050
 $Comp
 L Connector:Conn_01x03_Male J1
-U 1 1 60365C77
+U 1 1 603768FB
 P 2700 4700
 F 0 "J1" H 2672 4724 50  0000 R CNN
@@
 	-1   0    0    -1
 $EndComp
+Wire Wire Line
+	2150 4600 2500 4600
+Wire Wire Line
+	2150 4800 2500 4800
+Wire Wire Line
+	1700 4700 2500 4700
 $EndSCHEMATC

Commit message: update
Parts:
- R1, R2, R3, R4, R5: footprint Resistor_SMD:R_0603_1608Metric_Pad1.05x0.95mm_HandSolder -> Resistor_SMD:R_0603_1608Metric_Pad0.98x0.95mm_HandSolder
Changed lines of the file:
@@
 F 0 "R4" H 3009 3396 50  0000 L CNN
 F 1 "1.33K" H 3009 3305 50  0000 L CNN
-F 2 "Resistor_SMD:R_0603_1608Metric_Pad1.05x0.95mm_HandSolder" H 2950 3350 50  0001 C CNN
+F 2 "Resistor_SMD:R_0603_1608Metric_Pad0.98x0.95mm_HandSolder" H 2950 3350 50  0001 C CNN
 F 3 "~" H 2950 3350 50  0001 C CNN
 	1    2950 3350
@@
 F 0 "R3" H 2559 2546 50  0000 L CNN
 F 1 "20K" H 2559 2455 50  0000 L CNN
-F 2 "Resistor_SMD:R_0603_1608Metric_Pad1.05x0.95mm_HandSolder" H 2500 2500 50  0001 C CNN
+F 2 "Resistor_SMD:R_0603_1608Metric_Pad0.98x0.95mm_HandSolder" H 2500 2500 50  0001 C CNN
 F 3 "~" H 2500 2500 50  0001 C CNN
 	1    2500 2500
@@
 F 0 "R1" H 1759 4596 50  0000 L CNN
 F 1 "1K" H 1759 4505 50  0000 L CNN
-F 2 "Resistor_SMD:R_0603_1608Metric_Pad1.05x0.95mm_HandSolder" H 1700 4550 50  0001 C CNN
+F 2 "Resistor_SMD:R_0603_1608Metric_Pad0.98x0.95mm_HandSolder" H 1700 4550 50  0001 C CNN
 F 3 "~" H 1700 4550 50  0001 C CNN
 	1    1700 4550
@@
 F 0 "R2" H 1759 4896 50  0000 L CNN
 F 1 "150" H 1759 4805 50  0000 L CNN
-F 2 "Resistor_SMD:R_0603_1608Metric_Pad1.05x0.95mm_HandSolder" H 1700 4850 50  0001 C CNN
+F 2 "Resistor_SMD:R_0603_1608Metric_Pad0.98x0.95mm_HandSolder" H 1700 4850 50  0001 C CNN
 F 3 "~" H 1700 4850 50  0001 C CNN
 	1    1700 4850
@@
 F 0 "R5" V 5246 4550 50  0000 C CNN
 F 1 "300" V 5155 4550 50  0000 C CNN
-F 2 "Resistor_SMD:R_0603_1608Metric_Pad1.05x0.95mm_HandSolder" H 5050 4550 50  0001 C CNN
+F 2 "Resistor_SMD:R_0603_1608Metric_Pad0.98x0.95mm_HandSolder" H 5050 4550 50  0001 C CNN
 F 3 "~" H 5050 4550 50  0001 C CNN
 	1    5050 4550
