File: universal_power_board_v1.3/universal_power_board.kicad_pcb (KiCad board)
At the start: 2 copper layers, 41 x 41 mm, 25 parts, among them J1 Conn_01x03_Male, J10 5V OUTPUT, J11 BATT OUTPUT, J12 BATT OUTPUT, J2 BATT INPUT MAX14V, J3 BATT OUTPUT, J4 5V OUTPUT, J5 5V OUTPUT, J6 BATT OUTPUT, J7 5V OUTPUT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

Commit message: ステンシルデータ作成
Routing:
- net GND: vias 9 -> 15
Other:
- board text added: "UNIVERSAL POWER BOARD V1.4"
- board text removed: "UNIVERSAL POWER BOARD V1.3"
Changed lines of the file:
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@@
   (general
     (thickness 1.6)
-    (drawings 27)
-    (tracks 184)
+    (drawings 29)
+    (tracks 190)
     (zones 0)
     (modules 25)
@@
   (page A4)
   (layers
-    (0 F.Cu signal)
-    (31 B.Cu signal hide)
+    (0 F.Cu signal hide)
+    (31 B.Cu signal)
     (32 B.Adhes user)
     (33 F.Adhes user hide)
@@
     )
   )
+  (gr_poly (pts (xy 109.2454 89.0778) (xy 109.093 89.5604) (xy 109.093 89.5858) (xy 108.4326 90.0684) (xy 107.9246 89.789) (xy 107.823 89.7382) (xy 107.5182 89.662) (xy 107.2134 89.6874) (xy 106.9594 89.7636) (xy 106.4768 89.9414) (xy 106.68 88.8746) (xy 108.839 88.2396)) (layer B.Cu) (width 0.1))
+  (gr_poly (pts (xy 106.426 86.868) (xy 106.4006 91.3384) (xy 105.1814 91.3384) (xy 105.1814 86.7918) (xy 105.850055 86.03996)) (layer B.Cu) (width 0.1))
   (gr_text "+5V VOLT GND" (at 107.696 88.138) (layer F.SilkS)
     (effects (font (size 0.6 0.6) (thickness 0.125)))
@@
   )
   (gr_poly (pts (xy 108.01096 89.07018) (xy 106.82224 89.8144) (xy 106.02722 90.15984) (xy 105.67416 90.15222) (xy 105.70972 89.30132) (xy 106.81716 88.5317) (xy 108.01604 88.47328)) (layer B.Cu) (width 0.1))
-  (gr_poly (pts (xy 129.77622 65.06464) (xy 128.62814 67.10426) (xy 127.32766 67.13474) (xy 127.42418 65.73774) (xy 129.01422 64.87922)) (layer B.Cu) (width 0.1))
+  (gr_poly (pts (xy 130.59791 65.06972) (xy 129.85369 67.87388) (xy 127.3048 67.9704) (xy 127.42418 65.73774) (xy 129.01422 64.87922)) (layer B.Cu) (width 0.1))
   (gr_poly (pts (xy 129.37998 85.217) (xy 125.38456 85.12048) (xy 126.75362 67.89928) (xy 129.44348 65.74282)) (layer F.Cu) (width 0.1))
   (gr_poly (pts (xy 130.70332 64.94272) (xy 127.23876 68.48094) (xy 129.95148 71.4121) (xy 126.77902 74.60996) (xy 126.9492 75.67422) (xy 129.8067 78.55712) (xy 126.70536 81.75498) (xy 129.92862 85.2424) (xy 125.8824 85.46084) (xy 121.23166 90.42654) (xy 120.45696 90.30716) (xy 118.25224 88.24722) (xy 114.54638 88.34374) (xy 114.42446 90.7669) (xy 111.88192 88.32088) (xy 107.0356 88.44026) (xy 105.70464 90.06332) (xy 105.7275 88.32088) (xy 121.20626 87.9094) (xy 123.92152 85.14588) (xy 123.94438 78.14564) (xy 122.29846 76.54798) (xy 119.70512 76.42606) (xy 119.75338 72.08012) (xy 122.56516 71.9582) (xy 123.7742 70.47992) (xy 123.99264 67.7926) (xy 126.9492 64.8716)) (layer F.Cu) (width 0.1))
@@
   (gr_poly (pts (xy 129.02692 65.13576) (xy 127.72898 66.17716) (xy 125.4252 64.46266) (xy 127.39878 64.2747)) (layer B.Cu) (width 0.1))
   (gr_poly (pts (xy 120.94464 63.11138) (xy 112.50168 71.82104) (xy 106.4895 71.82104) (xy 106.59618 62.87008)) (layer B.Cu) (width 0.1))
-  (gr_text "UNIVERSAL POWER BOARD V1.3" (at 102.108 75.184 90) (layer F.SilkS)
+  (gr_text "UNIVERSAL POWER BOARD V1.4" (at 102.108 75.184 90) (layer F.SilkS)
     (effects (font (size 0.6 0.6) (thickness 0.125)))
   )
@@
   (segment (start 123.825 56.642) (end 104.648 56.642) (width 4) (layer F.Cu) (net 1))
   (segment (start 104.648 56.642) (end 123.825 56.642) (width 4) (layer B.Cu) (net 1))
+  (via (at 96.52 81.28) (size 0.8) (drill 0.4) (layers F.Cu B.Cu) (net 1))
+  (via (at 99.06 81.28) (size 0.8) (drill 0.4) (layers F.Cu B.Cu) (net 1))
+  (via (at 99.06 83.82) (size 0.8) (drill 0.4) (layers F.Cu B.Cu) (net 1))
+  (via (at 96.52 83.82) (size 0.8) (drill 0.4) (layers F.Cu B.Cu) (net 1))
+  (via (at 96.52 86.36) (size 0.8) (drill 0.4) (layers F.Cu B.Cu) (net 1))
+  (via (at 99.06 86.36) (size 0.8) (drill 0.4) (layers F.Cu B.Cu) (net 1))
   (via (at 102.87 66.04) (size 0.8) (drill 0.4) (layers F.Cu B.Cu) (net 2))
   (via (at 100.965 66.04) (size 0.8) (drill 0.4) (layers F.Cu B.Cu) (net 2))
